File: Button.kicad_sch (KiCad schematic)
At the start: 4 parts, among them SW1 TS02-66-43

Commit message: fixed wrong part number for tactile switches (leg length short -> long)
Parts:
- SW1: MOUSER# 179-TS026643BK100SCR -> 179-TS026643BK100LCR
Changed lines of the file:
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@@
 			)
 		)
-		(property "MOUSER#" "179-TS026643BK100SCR"
+		(property "MOUSER#" "179-TS026643BK100LCR"
 			(at 134.62 92.71 0)
 			(effects

Commit message: completed routing for revision 0.2
Parts:
- C10: footprint Capacitor_SMD:C_0603_1608Metric -> Capacitor_SMD:C_0805_2012Metric; MOUSER# 810-CGA3E2X7R1H104K -> 581-KGM21NR71H104KT
- R10: footprint Resistor_SMD:R_0402_1005Metric -> Resistor_SMD:R_0805_2012Metric; MOUSER# 603-RC0402FR-131KL -> 603-RC0805FR-101KL
- R11: footprint Resistor_SMD:R_0402_1005Metric -> Resistor_SMD:R_0805_2012Metric; MOUSER# 603-RE0402FRE0710KL -> 603-RC0805FR-7W10KL
Changed lines of the file:
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@@
 			)
 		)
-		(property "Footprint" "Resistor_SMD:R_0402_1005Metric"
+		(property "Footprint" "Resistor_SMD:R_0805_2012Metric"
 			(at 147.32 94.488 90)
 			(effects
@@
 			)
 		)
-		(property "MOUSER#" "603-RC0402FR-131KL"
+		(property "MOUSER#" "603-RC0805FR-101KL"
 			(at 147.32 92.71 0)
 			(effects
@@
 			)
 		)
-		(property "Footprint" "Resistor_SMD:R_0402_1005Metric"
+		(property "Footprint" "Resistor_SMD:R_0805_2012Metric"
 			(at 153.162 85.09 90)
 			(effects
@@
 			)
 		)
-		(property "MOUSER#" "603-RE0402FRE0710KL"
+		(property "MOUSER#" "603-RC0805FR-7W10KL"
 			(at 154.94 85.09 0)
 			(effects
@@
 			)
 		)
-		(property "Footprint" "Capacitor_SMD:C_0603_1608Metric"
+		(property "Footprint" "Capacitor_SMD:C_0805_2012Metric"
 			(at 155.9052 104.14 0)
 			(effects
@@
 			)
 		)
-		(property "MOUSER#" "810-CGA3E2X7R1H104K"
+		(property "MOUSER#" "581-KGM21NR71H104KT"
 			(at 154.94 100.33 0)
 			(effects

Commit message: added IDAnything
Parts:
- C10: IDAnything (none) -> 7306hr3vk0hr983c9yxsesf49q
- R10: IDAnything (none) -> f8p5h3y8kak8dbf84dv59qzqav
- R11: IDAnything (none) -> ct46g33j3jkr389e4bd4v5859v
- SW1: IDAnything (none) -> 5varex19v2jvwbnx5agzaw6w5v
Changed lines of the file:
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@@
+			)
+		)
+		(property "IDAnything" "f8p5h3y8kak8dbf84dv59qzqav"
+			(at 0 0 0)
+			(effects
+				(font
+					(size 1.27 1.27)
+				)
+				(hide yes)
 			)
 		)
@@
 			)
 		)
+		(property "IDAnything" "5varex19v2jvwbnx5agzaw6w5v"
+			(at 0 0 0)
+			(effects
+				(font
+					(size 1.27 1.27)
+				)
+				(hide yes)
+			)
+		)
 		(pin "1"
 		)
@@
 			)
 		)
+		(property "IDAnything" "ct46g33j3jkr389e4bd4v5859v"
+			(at 0 0 0)
+			(effects
+				(font
+					(size 1.27 1.27)
+				)
+				(hide yes)
+			)
+		)
 		(property "Height" ""
 			(at 154.94 85.09 0)
@@
 			(effects
 				(font
+					(size 1.27 1.27)
+				)
+				(hide yes)
+			)
+		)
+		(property "IDAnything" "7306hr3vk0hr983c9yxsesf49q"
+			(at 0 0 0)
+			(effects
+				(font
