File: DCDC.kicad_sch (KiCad schematic)
At the start: 12 parts, among them U2 LMR33620BDDA

Commit message: completed routing for revision 0.2
Parts:
- C4: footprint Capacitor_SMD:C_0603_1608Metric -> Capacitor_SMD:C_0805_2012Metric; MOUSER# 80-C0603C105K8PAC -> 187-CL21B105KAFNNNE
- C5, C9: footprint Capacitor_SMD:C_0603_1608Metric -> Capacitor_SMD:C_0805_2012Metric; MOUSER# 810-CGA3E2X7R1H104K -> 581-KGM21NR71H104KT
- C6: footprint Capacitor_SMD:C_0402_1005Metric -> Capacitor_SMD:C_0805_2012Metric; MOUSER# 963-UMK105CG330JV-F -> 80-C0805C330J5GACLR
- R8: footprint Resistor_SMD:R_0402_1005Metric -> Resistor_SMD:R_0805_2012Metric; MOUSER# 603-AC0402FR-13100KL -> 603-RE0805FRE07100KL
- R9: footprint Resistor_SMD:R_0402_1005Metric -> Resistor_SMD:R_0805_2012Metric; MOUSER# 667-ERJ-2RKF4322X -> 603-RC0805FR-0743K2L
Changed lines of the file:
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@@
 			)
 		)
-		(property "Footprint" "Capacitor_SMD:C_0603_1608Metric"
+		(property "Footprint" "Capacitor_SMD:C_0805_2012Metric"
 			(at 149.86 68.8848 0)
 			(effects
@@
 			)
 		)
-		(property "MOUSER#" "810-CGA3E2X7R1H104K"
+		(property "MOUSER#" "581-KGM21NR71H104KT"
 			(at 146.05 69.85 0)
 			(effects
@@
 			)
 		)
-		(property "Footprint" "Resistor_SMD:R_0402_1005Metric"
+		(property "Footprint" "Resistor_SMD:R_0805_2012Metric"
 			(at 181.102 96.52 90)
 			(effects
@@
 			)
 		)
-		(property "MOUSER#" "667-ERJ-2RKF4322X"
+		(property "MOUSER#" "603-RC0805FR-0743K2L"
 			(at 182.88 96.52 0)
 			(effects
@@
 			)
 		)
-		(property "Footprint" "Resistor_SMD:R_0402_1005Metric"
+		(property "Footprint" "Resistor_SMD:R_0805_2012Metric"
 			(at 181.102 83.82 90)
 			(effects
@@
 			)
 		)
-		(property "MOUSER#" "603-AC0402FR-13100KL"
+		(property "MOUSER#" "603-RE0805FRE07100KL"
 			(at 182.88 83.82 0)
 			(effects
@@
 			)
 		)
-		(property "Footprint" "Capacitor_SMD:C_0603_1608Metric"
+		(property "Footprint" "Capacitor_SMD:C_0805_2012Metric"
 			(at 112.7252 99.06 0)
 			(effects
@@
 			)
 		)
-		(property "MOUSER#" "80-C0603C105K8PAC"
+		(property "MOUSER#" "187-CL21B105KAFNNNE"
 			(at 111.76 95.25 0)
 			(effects
@@
 			)
 		)
-		(property "Footprint" "Capacitor_SMD:C_0603_1608Metric"
+		(property "Footprint" "Capacitor_SMD:C_0805_2012Metric"
 			(at 223.2152 93.98 0)
 			(effects
@@
 			)
 		)
-		(property "MOUSER#" "810-CGA3E2X7R1H104K"
+		(property "MOUSER#" "581-KGM21NR71H104KT"
 			(at 222.25 90.17 0)
 			(effects
@@
 			)
 		)
-		(property "Footprint" "Capacitor_SMD:C_0402_1005Metric"
+		(property "Footprint" "Capacitor_SMD:C_0805_2012Metric"
 			(at 172.4152 87.63 0)
 			(effects
@@
 			)
 		)
-		(property "MOUSER#" "963-UMK105CG330JV-F"
+		(property "MOUSER#" "80-C0805C330J5GACLR"
 			(at 171.45 83.82 0)
 			(effects

Commit message: completed silk screen
Parts:
- C2: MOUSER# 810-C3225X7R1H106MAC -> 810-C3225X7R1H106250
Changed lines of the file:
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@@
 			)
 		)
-		(property "MOUSER#" "810-C3225X7R1H106MAC"
+		(property "MOUSER#" "810-C3225X7R1H106250"
 			(at 83.82 88.9 0)
 			(effects

Commit message: added IDAnything
Parts:
- C2: IDAnything (none) -> 8ed1d4gh3rhtcap5n3thrqzk0z
- C3: IDAnything (none) -> 4a5rxdct54j399ddt59j5ethby
- C4: IDAnything (none) -> av0bek281wjtwa6a4nkznrfpj6
- C5, C9: IDAnything (none) -> 7306hr3vk0hr983c9yxsesf49q
- C6: IDAnything (none) -> 2rd8jddr1wjxzbs3sn3mevq907
- C7, C8: IDAnything (none) -> 5es6p5fr8rkjdahcs3x36hwzw2
- L1: IDAnything (none) -> 2hq8w74648jdvbnakgg56zq3m1
- R8: IDAnything (none) -> 4hwbycjybpjy48jy4908n6gzn6
- R9: IDAnything (none) -> 38cffz4qfmgyp8nxvts6531xbz
- U2: IDAnything (none) -> 7hxsg4786rhnabc7yv94snkhaf
Changed lines of the file:
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@@
+			)
+		)
+		(property "IDAnything" "7306hr3vk0hr983c9yxsesf49q"
+			(at 0 0 0)
+			(effects
+				(font
+					(size 1.27 1.27)
+				)
+				(hide yes)
 			)
 		)
@@
 			)
 		)
+		(property "IDAnything" "8ed1d4gh3rhtcap5n3thrqzk0z"
+			(at 0 0 0)
+			(effects
+				(font
+					(size 1.27 1.27)
+				)
+				(hide yes)
+			)
+		)
 		(pin "1"
 		)
@@
 			)
 		)
+		(property "IDAnything" "2hq8w74648jdvbnakgg56zq3m1"
+			(at 0 0 0)
+			(effects
+				(font
+					(size 1.27 1.27)
+				)
+				(hide yes)
+			)
+		)
 		(pin "2"
 		)
@@
 			)
 		)
+		(property "IDAnything" "7hxsg4786rhnabc7yv94snkhaf"
+			(at 0 0 0)
+			(effects
+				(font
+					(size 1.27 1.27)
+				)
+				(hide yes)
+			)
+		)
 		(pin "4"
 		)
@@
 			)
 		)
+		(property "IDAnything" "5es6p5fr8rkjdahcs3x36hwzw2"
+			(at 0 0 0)
+			(effects
+				(font
+					(size 1.27 1.27)
+				)
+				(hide yes)
+			)
+		)
 		(pin "1"
 		)
@@
 			)
 		)
+		(property "IDAnything" "38cffz4qfmgyp8nxvts6531xbz"
+			(at 0 0 0)
+			(effects
+				(font
+					(size 1.27 1.27)
+				)
+				(hide yes)
+			)
+		)
 		(pin "1"
 		)
@@
 			)
 		)
+		(property "IDAnything" "4hwbycjybpjy48jy4908n6gzn6"
+			(at 0 0 0)
+			(effects
+				(font
+					(size 1.27 1.27)
+				)
+				(hide yes)
+			)
+		)
 		(pin "1"
 		)
@@
 			)
 		)
+		(property "IDAnything" "4a5rxdct54j399ddt59j5ethby"
+			(at 0 0 0)
+			(effects
+				(font
+					(size 1.27 1.27)
+				)
+				(hide yes)
+			)
+		)
 		(pin "1"
 		)
@@
 			)
 		)
+		(property "IDAnything" "5es6p5fr8rkjdahcs3x36hwzw2"
+			(at 0 0 0)
+			(effects
+				(font
+					(size 1.27 1.27)
+				)
+				(hide yes)
+			)
+		)
 		(pin "1"
 		)
@@
 			)
 		)
+		(property "IDAnything" "av0bek281wjtwa6a4nkznrfpj6"
+			(at 0 0 0)
+			(effects
+				(font
+					(size 1.27 1.27)
+				)
+				(hide yes)
+			)
+		)
 		(pin "1"
 		)
@@
 		(property "MOUSER#" "581-KGM21NR71H104KT"
 			(at 222.25 90.17 0)
+			(effects
+				(font
+					(size 1.27 1.27)
+				)
+				(hide yes)
+			)
+		)
+		(property "IDAnything" "7306hr3vk0hr983c9yxsesf49q"
+			(at 0 0 0)
 			(effects
 				(font
@@
 			(effects
 				(font
+					(size 1.27 1.27)
+				)
+				(hide yes)
+			)
+		)
+		(property "IDAnything" "2rd8jddr1wjxzbs3sn3mevq907"
+			(at 0 0 0)
+			(effects
+				(font
